Commit message: added sim_mode argument

File: description/robot.urdf.xacro (robot description, xacro)
@@ -1,4 +1,6 @@
 <?xml version="1.0"?>
 <robot xmlns:xacro="http://www.ros.org/wiki/xacro"  name="robot">
+    <xacro:arg name="use_ros2_control" default="true"/>
+    <xacro:arg name="sim_mode" default="false"/>
     <xacro:include filename="robot_core.xacro" />
     <xacro:if value="$(arg use_ros2_control)">

File: description/ros2_control.xacro (robot description, xacro)
@@ -1,118 +1,118 @@
 <?xml version="1.0"?>
 <robot xmlns:xacro="http://www.ros.org/wiki/xacro">
-    <ros2_control name="RealRobot" type="system">
-        <hardware>
-            <plugin>carlikebot_ros2_control/CarlikeBotSystemHardware</plugin>
-            <param name="example_param_hw_start_duration_sec">0</param>
-            <param name="example_param_hw_stop_duration_sec">3.0</param>
-            <param name="front_left_wheel_joint_name">${prefix}front_left_wheel_joint</param>
-            <param name="front_right_wheel_joint_name">${prefix}front_right_wheel_joint</param>
-            <param name="rear_left_wheel_joint_name">${prefix}rear_left_wheel_joint</param>
-            <param name="rear_right_wheel_joint_name">${prefix}rear_right_wheel_joint</param>
-            <param name="loop_rate">30</param>
-            <param name="device">/dev/serial/by-path/platform-fd500000.pcie-pci-0000:01:00.0-usb-0:1.3:1.0-port0</param>
-            <param name="baud_rate">57600</param>
-            <param name="timeout_ms">2000</param>
-            <param name="enc_counts_per_rev_traction">4200</param>
-            <param name="enc_counts_per_rev_steering">4200</param>
-            <param name="pid_p">20</param>
-            <param name="pid_d">12</param>
-            <param name="pid_i">0</param>
-            <param name="pid_o">50</param>
-        </hardware>
-        <!-- Driving (traction) joints -->
-        <joint name="rear_left_wheel_joint">
-            <command_interface name="velocity"/>
-                <param name="min">-10</param>
-                <param name="max">10</param>
-            <state_interface name="velocity"/>
-            <state_interface name="position"/>
-        </joint>
-        <joint name="rear_right_wheel_joint">
-            <command_interface name="velocity"/>
-                <param name="min">-10</param>
-                <param name="max">10</param>
-            <state_interface name="velocity"/>
-            <state_interface name="position"/>
-        </joint>
-        <joint name="front_left_wheel_joint">
-            <command_interface name="velocity"/>
-                <param name="min">-10</param>
-                <param name="max">10</param>
-            <state_interface name="velocity"/>
-            <state_interface name="position"/>
-        </joint>
-        <joint name="front_right_wheel_joint">
-            <command_interface name="velocity"/>
-                <param name="min">-10</param>
-                <param name="max">10</param>
-            <state_interface name="velocity"/>
-            <state_interface name="position"/>
-        </joint>
-        <!-- Steering joints -->
-        <joint name="front_left_steering_joint">
-            <command_interface name="position"/>
-                <param name="min">-0.4</param>
-                <param name="max">0.4</param>
-            <state_interface name="velocity"/>
-            <state_interface name="position"/>
-        </joint>
-        <joint name="front_right_steering_joint">
-            <command_interface name="position"/>
-                <param name="min">-0.4</param>
-                <param name="max">0.4</param>
-            <state_interface name="velocity"/>
-            <state_interface name="position"/>
-        </joint>
-    </ros2_control>
-    <!-- <ros2_control name="GazeboSystem" type="system">
-        <hardware>
-            <plugin>gazebo_ros2_control/GazeboSystem</plugin>
-        </hardware>
-        <!-- Driving (traction) joints -->
-        <joint name="rear_left_wheel_joint">
-            <command_interface name="velocity"/>
-                <param name="min">-10</param>
-                <param name="max">10</param>
-            <state_interface name="velocity"/>
-            <state_interface name="position"/>
-        </joint>
-        <joint name="rear_right_wheel_joint">
-            <command_interface name="velocity"/>
-                <param name="min">-10</param>
-                <param name="max">10</param>
-            <state_interface name="velocity"/>
-            <state_interface name="position"/>
-        </joint>
-        <joint name="front_left_wheel_joint">
-            <command_interface name="velocity"/>
-                <param name="min">-10</param>
-                <param name="max">10</param>
-            <state_interface name="velocity"/>
-            <state_interface name="position"/>
-        </joint>
-        <joint name="front_right_wheel_joint">
-            <command_interface name="velocity"/>
-                <param name="min">-10</param>
-                <param name="max">10</param>
-            <state_interface name="velocity"/>
-            <state_interface name="position"/>
-        </joint>
-        <!-- Steering joints -->
-        <joint name="front_left_steering_joint">
-            <command_interface name="position"/>
-                <param name="min">-0.4</param>
-                <param name="max">0.4</param>
-            <state_interface name="velocity"/>
-            <state_interface name="position"/>
-        </joint>
-        <joint name="front_right_steering_joint">
-            <command_interface name="position"/>
-                <param name="min">-0.4</param>
-                <param name="max">0.4</param>
-            <state_interface name="velocity"/>
-            <state_interface name="position"/>
-        </joint>
-    </ros2_control> -->
+    <xacro:unless value="$(arg sim_mode)">
+        <ros2_control name="RealRobot" type="system">
+            <hardware>
+                <plugin>carlikebot_ros2_control/CarlikeBotSystemHardware</plugin>
+                <param name="example_param_hw_start_duration_sec">0</param>
+                <param name="example_param_hw_stop_duration_sec">3.0</param>
+                <param name="front_left_wheel_joint_name">${prefix}front_left_wheel_joint</param>
+                <param name="front_right_wheel_joint_name">${prefix}front_right_wheel_joint</param>
+                <param name="rear_left_wheel_joint_name">${prefix}rear_left_wheel_joint</param>
+                <param name="rear_right_wheel_joint_name">${prefix}rear_right_wheel_joint</param>
+                <param name="loop_rate">30</param>
+                <param name="device">/dev/serial/by-path/platform-fd500000.pcie-pci-0000:01:00.0-usb-0:1.3:1.0-port0</param>
+                <param name="baud_rate">57600</param>
+                <param name="timeout_ms">2000</param>
+                <param name="enc_counts_per_rev_traction">4200</param>
+                <param name="enc_counts_per_rev_steering">4200</param>
+                <param name="pid_p">20</param>
+                <param name="pid_d">12</param>
+                <param name="pid_i">0</param>
+                <param name="pid_o">50</param>
+            </hardware>
+            <!-- Driving (traction) joints -->
+            <joint name="rear_left_wheel_joint">
+                <command_interface name="velocity"/>
+                    <param name="min">-10</param>
+                    <param name="max">10</param>
+                <state_interface name="velocity"/>
+                <state_interface name="position"/>
+            </joint>
+            <joint name="rear_right_wheel_joint">
+                <command_interface name="velocity"/>
+                    <param name="min">-10</param>
+                    <param name="max">10</param>
+                <state_interface name="velocity"/>
+                <state_interface name="position"/>
+            </joint>
+            <!-- <joint name="front_left_wheel_joint">
+                <command_interface name="velocity"/>
+                    <param name="min">-10</param>
+                    <param name="max">10</param>
+                <state_interface name="velocity"/>
+                <state_interface name="position"/>
+            </joint>
+            <joint name="front_right_wheel_joint">
+                <command_interface name="velocity"/>
+                    <param name="min">-10</param>
+                    <param name="max">10</param>
+                <state_interface name="velocity"/>
+                <state_interface name="position"/>
+            </joint>  -->
+            <!-- Steering joints -->
+            <joint name="front_left_steering_joint">
+                <command_interface name="position"/>
+                    <param name="min">-0.4</param>
+                    <param name="max">0.4</param>
+                <state_interface name="position"/>
+            </joint>
+            <joint name="front_right_steering_joint">
+                <command_interface name="position"/>
+                    <param name="min">-0.4</param>
+                    <param name="max">0.4</param>
+                <state_interface name="position"/>
+            </joint>
+        </ros2_control>
+    </xacro:unless>
+    <xacro:if value="$(arg sim_mode)">
+        <ros2_control name="GazeboSystem" type="system">
+            <hardware>
+                <plugin>gazebo_ros2_control/GazeboSystem</plugin>
+            </hardware>
+            <!-- Driving (traction) joints -->
+            <joint name="rear_left_wheel_joint">
+                <command_interface name="velocity"/>
+                    <param name="min">-10</param>
+                    <param name="max">10</param>
+                <state_interface name="velocity"/>
+                <state_interface name="position"/>
+            </joint>
+            <joint name="rear_right_wheel_joint">
+                <command_interface name="velocity"/>
+                    <param name="min">-10</param>
+                    <param name="max">10</param>
+                <state_interface name="velocity"/>
+                <state_interface name="position"/>
+            </joint>
+            <joint name="front_left_wheel_joint">
+                <command_interface name="velocity"/>
+                    <param name="min">-10</param>
+                    <param name="max">10</param>
+                <state_interface name="velocity"/>
+                <state_interface name="position"/>
+            </joint>
+            <joint name="front_right_wheel_joint">
+                <command_interface name="velocity"/>
+                    <param name="min">-10</param>
+                    <param name="max">10</param>
+                <state_interface name="velocity"/>
+                <state_interface name="position"/>
+            </joint>
+            <!-- Steering joints -->
+            <joint name="front_left_steering_joint">
+                <command_interface name="position"/>
+                    <param name="min">-0.4</param>
+                    <param name="max">0.4</param>
+                <state_interface name="position"/>
+            </joint>
+            <joint name="front_right_steering_joint">
+                <command_interface name="position"/>
+                    <param name="min">-0.4</param>
+                    <param name="max">0.4</param>
+                <state_interface name="position"/>
+            </joint>
+        </ros2_control>
+    </xacro:if>
     <gazebo>
         <plugin name="gazebo_ros2_control" filename="libgazebo_ros2_control.so">
@@ -123,4 +123,5 @@
             </ros>
             <parameters>$(find seav2)/config/my_controllers.yaml</parameters>
+            <parameters>$(find seav2)/config/gaz_ros2_ctl_use_sim.yaml</parameters>
         </plugin>
     </gazebo>
