Commit message: fixed laser frame tf

File: description/lidar.xacro (robot description, xacro)
@@ -1,10 +1,10 @@
 <?xml version="1.0"?>
 <robot xmlns:xacro="http://www.ros.org/wiki/xacro"  name="robot">
-    <joint name="lidar_joint" type="fixed">
+    <joint name="laser_joint" type="fixed">
         <parent link="chassis"/>
-        <child link="lidar_frame"/>
+        <child link="laser_frame"/>
         <origin xyz="-0.2 0 0.15" rpy="0 0 0"/>
     </joint>
-    <link name="lidar_frame">
+    <link name="laser_frame">
         <visual>
             <geometry>
@@ -22,7 +22,7 @@
         </xacro:inertial_cylinder>
     </link>
-    <gazebo reference="lidar_frame">
+    <gazebo reference="laser_frame">
         <material>Gazebo/Blue</material>
-        <sensor name="lidar" type="ray">
+        <sensor name="laser" type="ray">
             <pose> 0 0 0 0 0 0 </pose>
             <visualize>true</visualize>
@@ -41,10 +41,10 @@
                 </range>
             </ray>
-            <plugin name="lidar_controller" filename="libgazebo_ros_ray_sensor.so">
+            <plugin name="laser_controller" filename="libgazebo_ros_ray_sensor.so">
                 <ros>
                     <argument>~/out:=scan</argument>
                 </ros>
                 <output_type>sensor_msgs/LaserScan</output_type>
-                <frame_name>lidar_frame</frame_name>
+                <frame_name>laser_frame</frame_name>
             </plugin>
         </sensor>
