Commit message: fix URDF steering joints

File: description/robot_core.xacro (robot description, xacro)
@@ -60,5 +60,5 @@
         <parent link="chassis"/>
         <child link="left_steering_link"/>
-        <origin xyz="0.3 0.17 0" rpy="0 0 0"/>
+        <origin xyz="0.3 0.21 0" rpy="0 0 0"/>
         <axis xyz="0 0 1"/>
         <limit lower="-${pi/8}" upper="${pi/8}" effort="20" velocity="5"/> <!-- TODO -->
@@ -73,5 +73,5 @@
         <parent link="left_steering_link"/>
         <child link="front_left_wheel"/>
-        <origin xyz="0 0.04 0" rpy="${pi/2} 0 0"/>
+        <origin xyz="0 0 0" rpy="${pi/2} 0 0"/>
         <axis xyz="0 0 -1"/>
         <dynamics friction="0.8" damping="0.5" /> <!-- TODO -->
@@ -106,5 +106,5 @@
         <parent link="chassis"/>
         <child link="right_steering_link"/>
-        <origin xyz="0.3 -0.17 0" rpy="0 0 0"/>
+        <origin xyz="0.3 -0.21 0" rpy="0 0 0"/>
         <axis xyz="0 0 1"/>
         <limit lower="-${pi/8}" upper="${pi/8}" effort="20" velocity="5"/> <!-- TODO -->
@@ -119,5 +119,5 @@
         <parent link="right_steering_link"/>
         <child link="front_right_wheel"/>
-        <origin xyz="0 -0.04 0" rpy="-${pi/2} 0 0"/>
+        <origin xyz="0 0 0" rpy="-${pi/2} 0 0"/>
         <axis xyz="0 0 1"/>
         <dynamics friction="0.8" damping="0.5" /> <!-- TODO -->

Commit message: added Lidar sim

File: description/robot_core.xacro (robot description, xacro)
@@ -15,10 +15,14 @@
     </material>
     <!-- BASE FOOTPRINT LINK -->
-    <link name="base_footprint">
+    <!-- <joint name="footprint_joint" type="fixed">
+        <child link="footprint_link" />
+        <origin xyz="0 0 0" rpy="0 0 0" />
+    </joint> -->
+    <link name="footprint_link">
         <origin xyz="0 0 0" rpy="0 0 0" />
     </link>
     <!-- BASE LINK -->
     <joint name="base_joint" type="fixed">
-        <parent link="base_footprint" />
+        <parent link="footprint_link" />
         <child link="base_link" />
         <origin xyz="-0.3 0.0 0.1" rpy="0 0 0" />

Commit message: fixed odom frame and tree

File: description/robot_core.xacro (robot description, xacro)
@@ -14,18 +14,19 @@
         <color rgba="0 0 0 1"/>
     </material>
-    <!-- BASE FOOTPRINT LINK -->
-    <!-- <joint name="footprint_joint" type="fixed">
+    <!-- BASE LINK -->
+    <!-- <joint name="base_joint" type="fixed">
+        <parent link="world"/>
+        <child link="base_link" />
+        <origin xyz="-0.3 0.0 0.1" rpy="0 0 0" />
+    </joint> -->
+    <link name="base_link">
+    </link>
+    <!-- FOOTPRINT LINK -->
+    <joint name="footprint_joint" type="fixed">
+        <parent link="base_link" />
         <child link="footprint_link" />
         <origin xyz="0 0 0" rpy="0 0 0" />
-    </joint> -->
+    </joint>
     <link name="footprint_link">
-    </link>
-    <!-- BASE LINK -->
-    <joint name="base_joint" type="fixed">
-        <parent link="footprint_link" />
-        <child link="base_link" />
-        <origin xyz="-0.3 0.0 0.1" rpy="0 0 0" />
-    </joint>
-    <link name="base_link">
     </link>
     <!-- CHASSIS LINK -->
@@ -60,26 +61,12 @@
     <joint name="front_left_steering_joint" type="revolute">
         <parent link="base_link"/>
-        <child link="left_steering_link"/>
+        <child link="front_left_wheel"/>
         <origin xyz="0.6 0.21 0" rpy="0 0 0"/>
         <axis xyz="0 0 1"/>
-        <limit lower="-${pi/8}" upper="${pi/8}" effort="20" velocity="5"/> <!-- TODO -->
-    </joint>
-    <link name="left_steering_link">
-        <xacro:inertial_cylinder mass="0.01" radius="0.1" length="0.08">
-            <origin xyz="0 0 0" rpy="0 0 0"/>
-        </xacro:inertial_cylinder>
-    </link>
-    <!-- rotation -->
-    <joint name="front_left_wheel_joint" type="continuous">
-        <parent link="left_steering_link"/>
-        <child link="front_left_wheel"/>
-        <origin xyz="0 0 0" rpy="${pi/2} 0 0"/>
-        <axis xyz="0 0 -1"/>
-        <dynamics friction="0.8" damping="0.5" /> <!-- TODO -->
-        <limit lower="-3.14159" upper="3.14159" effort="0" velocity="1" /> <!-- TODO -->
+        <limit lower="-${pi/8}" upper="${pi/8}" effort="20" velocity="5"/>
     </joint>
     <link name="front_left_wheel">
         <visual>
-            <origin xyz="0 0 0" rpy="0 0 0"/>
+            <origin xyz="0 0 0" rpy="${pi/2} 0 0"/>
             <geometry>
                 <cylinder radius="0.1" length="0.08"/>
@@ -99,6 +86,6 @@
     <gazebo reference="front_left_wheel">
         <material>Gazebo/Black</material>
-        <mu1>5</mu1> <!-- TODO -->
-        <mu2>5</mu2> <!-- TODO -->
+        <mu1>5</mu1>
+        <mu2>5</mu2>
     </gazebo>
     <!-- FRONT RIGHT WHEEL -->
@@ -106,26 +93,12 @@
     <joint name="front_right_steering_joint" type="revolute">
         <parent link="base_link"/>
-        <child link="right_steering_link"/>
+        <child link="front_right_wheel"/>
         <origin xyz="0.6 -0.21 0" rpy="0 0 0"/>
         <axis xyz="0 0 1"/>
-        <limit lower="-${pi/8}" upper="${pi/8}" effort="20" velocity="5"/> <!-- TODO -->
-    </joint>
-    <link name="right_steering_link">
-        <xacro:inertial_cylinder mass="0.01" radius="0.1" length="0.08">
-            <origin xyz="0 0 0" rpy="0 0 0"/>
-        </xacro:inertial_cylinder>
-    </link>
-    <!-- rotation -->
-    <joint name="front_right_wheel_joint" type="continuous">
-        <parent link="right_steering_link"/>
-        <child link="front_right_wheel"/>
-        <origin xyz="0 0 0" rpy="-${pi/2} 0 0"/>
-        <axis xyz="0 0 1"/>
-        <dynamics friction="0.8" damping="0.5" /> <!-- TODO -->
-        <limit lower="-3.14159" upper="3.14159" effort="0" velocity="1" /> <!-- TODO -->
+        <limit lower="-${pi/8}" upper="${pi/8}" effort="20" velocity="5"/>
     </joint>
     <link name="front_right_wheel">
         <visual>
-            <origin xyz="0 0 0" rpy="0 0 0"/>
+            <origin xyz="0 0 0" rpy="-${pi/2} 0 0"/>
             <geometry>
                 <cylinder radius="0.1" length="0.08"/>
@@ -145,6 +118,6 @@
     <gazebo reference="front_right_wheel">
         <material>Gazebo/Black</material>
-        <mu1>5</mu1> <!-- TODO -->
-        <mu2>5</mu2> <!-- TODO -->
+        <mu1>5</mu1>
+        <mu2>5</mu2>
     </gazebo>
     <!-- REAR LEFT WHEEL -->
@@ -155,6 +128,6 @@
         <origin xyz="0 0.21 0" rpy="${pi/2} 0 0"/>
         <axis xyz="0 0 -1"/>
-        <dynamics friction="0.8" damping="0.5" /> <!-- TODO -->
-        <limit lower="-3.14159" upper="3.14159" effort="200" velocity="1" /> <!-- TODO -->
+        <dynamics friction="0.8" damping="0.5" />
+        <limit lower="-3.14159" upper="3.14159" effort="200" velocity="1" />
     </joint>
     <link name="rear_left_wheel">
@@ -178,6 +151,6 @@
     <gazebo reference="rear_left_wheel">
         <material>Gazebo/Black</material>
-        <mu1>10</mu1> <!-- TODO -->
-        <mu2>10</mu2> <!-- TODO -->
+        <mu1>10</mu1>
+        <mu2>10</mu2>
     </gazebo>
     <!-- REAR RIGHT WHEEL -->
@@ -188,6 +161,6 @@
         <origin xyz="0 -0.21 0" rpy="-${pi/2} 0 0"/>
         <axis xyz="0 0 1"/>
-        <dynamics friction="0.8" damping="0.5" /> <!-- TODO -->
-        <limit lower="-3.14159" upper="3.14159" effort="200" velocity="1" /> <!-- TODO -->
+        <dynamics friction="0.8" damping="0.5" />
+        <limit lower="-3.14159" upper="3.14159" effort="200" velocity="1" />
     </joint>
     <link name="rear_right_wheel">
@@ -211,6 +184,6 @@
     <gazebo reference="rear_right_wheel">
         <material>Gazebo/Black</material>
-        <mu1>10</mu1> <!-- TODO -->
-        <mu2>10</mu2> <!-- TODO -->
+        <mu1>10</mu1>
+        <mu2>10</mu2>
     </gazebo>
     <!-- VIRTUAL STEERING WHEEL -->

Commit message: got SLAM working

File: description/robot_core.xacro (robot description, xacro)
@@ -23,10 +23,10 @@
     </link>
     <!-- FOOTPRINT LINK -->
-    <joint name="footprint_joint" type="fixed">
+    <joint name="base_footprint_joint" type="fixed">
         <parent link="base_link" />
-        <child link="footprint_link" />
-        <origin xyz="0 0 0" rpy="0 0 0" />
-    </joint>
-    <link name="footprint_link">
+        <child link="base_footprint" />
+        <origin xyz="-0.1 0 0" rpy="0 0 0" />
+    </joint>
+    <link name="base_footprint">
     </link>
     <!-- CHASSIS LINK -->

File: description/ros2_control.xacro (robot description, xacro)
@@ -15,6 +15,6 @@
                 <param name="baud_rate">57600</param>
                 <param name="timeout_ms">2000</param>
-                <param name="enc_counts_per_rev_traction">4200</param>
-                <param name="enc_counts_per_rev_steering">4200</param>
+                <param name="enc_counts_per_rev_traction">210</param>
+                <param name="enc_counts_per_rev_steering">25</param>
                 <param name="pid_p">20</param>
                 <param name="pid_d">12</param>

Commit message: fixed front wheel sim collision

File: description/robot_core.xacro (robot description, xacro)
@@ -75,5 +75,5 @@
         </visual>
         <collision>
-            <origin xyz="0 0 0" rpy="0 0 0"/>
+            <origin xyz="0 0 0" rpy="${pi/2} 0 0"/>
             <geometry>
                 <cylinder radius="0.1" length="0.08"/>
@@ -107,5 +107,5 @@
         </visual>
         <collision>
-            <origin xyz="0 0 0" rpy="0 0 0"/>
+            <origin xyz="0 0 0" rpy="-${pi/2} 0 0"/>
             <geometry>
                 <cylinder radius="0.1" length="0.08"/>

Commit message: fixed urdf for gaz sim

File: description/robot_core.xacro (robot description, xacro)
@@ -61,19 +61,33 @@
     <joint name="front_left_steering_joint" type="revolute">
         <parent link="base_link"/>
-        <child link="front_left_wheel"/>
+        <child link="front_left_steering_link"/>
         <origin xyz="0.6 0.21 0" rpy="0 0 0"/>
         <axis xyz="0 0 1"/>
         <limit lower="-${pi/8}" upper="${pi/8}" effort="20" velocity="5"/>
     </joint>
+    <link name="front_left_steering_link">
+        <xacro:inertial_cylinder mass="0.01" radius="0.1" length="0.08">
+            <origin xyz="0 0 0" rpy="${pi/2} 0 0"/>
+        </xacro:inertial_cylinder>
+    </link>
+    <!-- rotation -->
+    <joint name="front_left_wheel_joint" type="continuous">
+        <parent link="front_left_steering_link"/>
+        <child link="front_left_wheel"/>
+        <origin xyz="0 0 0" rpy="${pi/2} 0 0"/>
+        <axis xyz="0 0 -1"/>
+        <dynamics friction="0.8" damping="0.5" /> <!-- TODO -->
+        <limit lower="-3.14159" upper="3.14159" effort="0" velocity="1" /> <!-- TODO -->
+    </joint>
     <link name="front_left_wheel">
         <visual>
-            <origin xyz="0 0 0" rpy="${pi/2} 0 0"/>
-            <geometry>
-                <cylinder radius="0.1" length="0.08"/>
-            </geometry>
-            <material name="black"/>
-        </visual>
-        <collision>
-            <origin xyz="0 0 0" rpy="${pi/2} 0 0"/>
+            <origin xyz="0 0 0" rpy="0 0 0"/>
+            <geometry>
+                <cylinder radius="0.1" length="0.08"/>
+            </geometry>
+            <material name="black"/>
+        </visual>
+        <collision>
+            <origin xyz="0 0 0" rpy="0 0 0"/>
             <geometry>
                 <cylinder radius="0.1" length="0.08"/>
@@ -93,19 +107,33 @@
     <joint name="front_right_steering_joint" type="revolute">
         <parent link="base_link"/>
-        <child link="front_right_wheel"/>
+        <child link="front_right_steering_link"/>
         <origin xyz="0.6 -0.21 0" rpy="0 0 0"/>
         <axis xyz="0 0 1"/>
         <limit lower="-${pi/8}" upper="${pi/8}" effort="20" velocity="5"/>
     </joint>
+    <link name="front_right_steering_link">
+        <xacro:inertial_cylinder mass="0.01" radius="0.1" length="0.08">
+            <origin xyz="0 0 0" rpy="${pi/2} 0 0"/>
+        </xacro:inertial_cylinder>
+    </link>
+    <!-- rotation -->
+    <joint name="front_right_wheel_joint" type="continuous">
+        <parent link="front_right_steering_link"/>
+        <child link="front_right_wheel"/>
+        <origin xyz="0 0 0" rpy="${pi/2} 0 0"/>
+        <axis xyz="0 0 -1"/>
+        <dynamics friction="0.8" damping="0.5" /> <!-- TODO -->
+        <limit lower="-3.14159" upper="3.14159" effort="0" velocity="1" /> <!-- TODO -->
+    </joint>
     <link name="front_right_wheel">
         <visual>
-            <origin xyz="0 0 0" rpy="-${pi/2} 0 0"/>
-            <geometry>
-                <cylinder radius="0.1" length="0.08"/>
-            </geometry>
-            <material name="black"/>
-        </visual>
-        <collision>
-            <origin xyz="0 0 0" rpy="-${pi/2} 0 0"/>
+            <origin xyz="0 0 0" rpy="0 0 0"/>
+            <geometry>
+                <cylinder radius="0.1" length="0.08"/>
+            </geometry>
+            <material name="black"/>
+        </visual>
+        <collision>
+            <origin xyz="0 0 0" rpy="0 0 0"/>
             <geometry>
                 <cylinder radius="0.1" length="0.08"/>
