Commit message: added real robot launch file

File: description/ros2_control.xacro (robot description, xacro)
@@ -1,5 +1,70 @@
 <?xml version="1.0"?>
 <robot xmlns:xacro="http://www.ros.org/wiki/xacro">
-    <ros2_control name="GazeboSystem" type="system">
+    <ros2_control name="RealRobot" type="system">
+        <hardware>
+            <plugin>carlikebot_ros2_control/CarlikeBotSystemHardware</plugin>
+            <param name="example_param_hw_start_duration_sec">0</param>
+            <param name="example_param_hw_stop_duration_sec">3.0</param>
+            <param name="front_left_wheel_joint_name">${prefix}front_left_wheel_joint</param>
+            <param name="front_right_wheel_joint_name">${prefix}front_right_wheel_joint</param>
+            <param name="rear_left_wheel_joint_name">${prefix}rear_left_wheel_joint</param>
+            <param name="rear_right_wheel_joint_name">${prefix}rear_right_wheel_joint</param>
+            <param name="loop_rate">30</param>
+            <param name="device">/dev/serial/by-path/platform-fd500000.pcie-pci-0000:01:00.0-usb-0:1.3:1.0-port0</param>
+            <param name="baud_rate">57600</param>
+            <param name="timeout_ms">2000</param>
+            <param name="enc_counts_per_rev_traction">4200</param>
+            <param name="enc_counts_per_rev_steering">4200</param>
+            <param name="pid_p">20</param>
+            <param name="pid_d">12</param>
+            <param name="pid_i">0</param>
+            <param name="pid_o">50</param>
+        </hardware>
+        <!-- Driving (traction) joints -->
+        <joint name="rear_left_wheel_joint">
+            <command_interface name="velocity"/>
+                <param name="min">-10</param>
+                <param name="max">10</param>
+            <state_interface name="velocity"/>
+            <state_interface name="position"/>
+        </joint>
+        <joint name="rear_right_wheel_joint">
+            <command_interface name="velocity"/>
+                <param name="min">-10</param>
+                <param name="max">10</param>
+            <state_interface name="velocity"/>
+            <state_interface name="position"/>
+        </joint>
+        <joint name="front_left_wheel_joint">
+            <command_interface name="velocity"/>
+                <param name="min">-10</param>
+                <param name="max">10</param>
+            <state_interface name="velocity"/>
+            <state_interface name="position"/>
+        </joint>
+        <joint name="front_right_wheel_joint">
+            <command_interface name="velocity"/>
+                <param name="min">-10</param>
+                <param name="max">10</param>
+            <state_interface name="velocity"/>
+            <state_interface name="position"/>
+        </joint>
+        <!-- Steering joints -->
+        <joint name="front_left_steering_joint">
+            <command_interface name="position"/>
+                <param name="min">-0.4</param>
+                <param name="max">0.4</param>
+            <state_interface name="velocity"/>
+            <state_interface name="position"/>
+        </joint>
+        <joint name="front_right_steering_joint">
+            <command_interface name="position"/>
+                <param name="min">-0.4</param>
+                <param name="max">0.4</param>
+            <state_interface name="velocity"/>
+            <state_interface name="position"/>
+        </joint>
+    </ros2_control>
+    <!-- <ros2_control name="GazeboSystem" type="system">
         <hardware>
             <plugin>gazebo_ros2_control/GazeboSystem</plugin>
@@ -49,5 +114,5 @@
             <state_interface name="position"/>
         </joint>
-    </ros2_control>
+    </ros2_control> -->
     <gazebo>
         <plugin name="gazebo_ros2_control" filename="libgazebo_ros2_control.so">

Commit message: front traction state interfaces

File: description/ros2_control.xacro (robot description, xacro)
@@ -37,18 +37,12 @@
                 <state_interface name="position"/>
             </joint>
-            <!-- <joint name="front_left_wheel_joint">
-                <command_interface name="velocity"/>
-                    <param name="min">-10</param>
-                    <param name="max">10</param>
+            <joint name="front_left_wheel_joint">
                 <state_interface name="velocity"/>
                 <state_interface name="position"/>
             </joint>
             <joint name="front_right_wheel_joint">
-                <command_interface name="velocity"/>
-                    <param name="min">-10</param>
-                    <param name="max">10</param>
                 <state_interface name="velocity"/>
                 <state_interface name="position"/>
-            </joint>  -->
+            </joint>
             <!-- Steering joints -->
             <joint name="front_left_steering_joint">
